File: Hardware/SparkFun Qwiic ToF Imager - VL53L5CX.sch (EAGLE design)
At the start: 36 parts, among them J3 PTH, U1 VL53L5CX

Commit message: Reduce copper and paste aperatures on VL53L5CX FP.
Changed lines of the file:
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@@
 <part name="R4" library="SparkFun-Resistors" deviceset="2.2KOHM" device="-0603-1/10W-1%" value="2.2k"/>
 <part name="R5" library="SparkFun-Resistors" deviceset="2.2KOHM" device="-0603-1/10W-1%" value="2.2k"/>
-<part name="I2C" library="SparkFun-Jumpers" deviceset="JUMPER-SMT_3_2-NC_TRACE" device="_SILK" package3d_urn="urn:adsk.eagle:package:39289/1" value=""/>
+<part name="I2C" library="SparkFun-Jumpers" deviceset="JUMPER-SMT_3_2-NC_TRACE" device="_SILK" package3d_urn="urn:adsk.eagle:package:39289/1" value="JUMPER-SMT_3_2-NC_TRACE_SILK"/>
 <part name="SUPPLY4" library="SparkFun-PowerSymbols" deviceset="3.3V" device=""/>
 <part name="J2" library="SparkFun-Connectors" deviceset="QWIIC_CONNECTOR" device="JS-1MM"/>

Commit message: Fix I2C address in schematic.
Other:
- note added: "7-bit unshifted I2C address: 0x29"
- note removed: "7-bit unshifted I2C address: 0x52"
Changed lines of the file:
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@@
 <text x="170.434" y="11.43" size="2.54" layer="94" font="vector">N. Seidle</text>
 <text x="237.744" y="7.366" size="2.54" layer="94" font="vector">v10</text>
-<text x="121.92" y="111.76" size="1.778" layer="97" font="vector" align="center">7-bit unshifted I2C address: 0x52</text>
+<text x="121.92" y="111.76" size="1.778" layer="97" font="vector" align="center">7-bit unshifted I2C address: 0x29</text>
 <text x="193.04" y="157.48" size="1.778" layer="97" font="vector" align="center">Cut I²C jumper to
 remove pull-ups from bus</text>
@@
 <instance part="I2C" gate="G$1" x="172.72" y="149.86" smashed="yes" rot="R270">
 <attribute name="NAME" x="170.942" y="146.05" size="1.778" layer="95" font="vector"/>
-<attribute name="VALUE" x="172.339" y="147.32" size="1.778" layer="96" font="vector" rot="R270" align="top-left"/>
 </instance>
 <instance part="SUPPLY4" gate="G$1" x="50.8" y="66.04" smashed="yes">
