File: Hardware/Production/SparkFun Qwiic ToF Imager - VL53L5CX-Panel.brd (EAGLE design)
At the start: 175 x 117.3 mm, 1494 parts, among them J10 PTH, J106 PTH, J114 PTH, J122 PTH, J130 PTH, J138 PTH, J146 PTH, J154 PTH, J162 PTH, J170 PTH, J178 PTH, J18 PTH, J186 PTH, J26 PTH, J3 PTH, J34 PTH, J42 PTH, J50 PTH, J58 PTH, J66 PTH, J74 PTH, J82 PTH, J90 PTH, J98 PTH, U1 VL53L5CX, U10 VL53L5CX, U11 VL53L5CX, U12 VL53L5CX, U13 VL53L5CX, U14 VL53L5CX, U15 VL53L5CX, U16 VL53L5CX, U17 VL53L5CX, U18 VL53L5CX, U19 VL53L5CX, U2 VL53L5CX, U20 VL53L5CX, U21 VL53L5CX, U22 VL53L5CX, U23 VL53L5CX, U24 VL53L5CX, U3 VL53L5CX, U4 VL53L5CX, U5 VL53L5CX, U6 VL53L5CX, U7 VL53L5CX, U8 VL53L5CX, U9 VL53L5CX

Commit message: Add production files post design review
Parts:
- JP108, JP119, JP130, JP141, JP152, JP163, JP174, JP185, JP196, JP20, JP207, JP218, JP229, JP240, JP251, JP262, JP31, JP42, JP53, JP64, JP75, JP8, JP86, JP97: value (none) -> PSU
Routing:
- net N$99: track 12.0 -> 9.91 mm
- net N$93: track 12.0 -> 9.91 mm
- net N$135: track 12.0 -> 9.91 mm
- net N$129: track 12.0 -> 9.91 mm
- net N$141: track 12.0 -> 9.91 mm
- net N$105: track 12.0 -> 9.91 mm
- net N$27: track 12.0 -> 9.91 mm
- net N$21: track 12.0 -> 9.91 mm
- net N$33: track 12.0 -> 9.91 mm
- net N$63: track 12.0 -> 9.91 mm
- net N$57: track 12.0 -> 9.91 mm
- net N$81: track 12.0 -> 9.91 mm
- net N$117: track 12.0 -> 9.91 mm
- net N$87: track 12.0 -> 9.91 mm
- net N$123: track 12.0 -> 9.91 mm
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
Commit message: Reduce copper and paste aperatures on VL53L5CX FP.
Parts:
- I2C, I2C1, I2C10, I2C11, I2C12, I2C13, I2C14, I2C15, I2C16, I2C17, I2C18, I2C19, I2C2, I2C20, I2C21, I2C22, I2C23, I2C3, I2C4, I2C5, I2C6, I2C7, I2C8, I2C9: value (none) -> JUMPER-SMT_3_2-NC_TRACE_SILK
Other:
- board text added: "v11"
- board text removed: "v10"

Commit message: Add panel files for v1.1
Parts:
- U$100, U$129, U$158, U$187, U$216, U$245, U$274, U$303, U$332, U$361, U$390, U$419, U$42, U$448, U$477, U$506, U$535, U$564, U$593, U$622, U$651, U$680, U$71: device output:#RST#1 -> output:#INT_#0
- U$101, U$130, U$159, U$188, U$217, U$246, U$275, U$304, U$333, U$362, U$391, U$420, U$43, U$449, U$478, U$507, U$536, U$565, U$594, U$623, U$652, U$681, U$72: device output:#INT_#0 -> output:#RST_#1
- U$102, U$131, U$160, U$189, U$218, U$247, U$276, U$305, U$334, U$363, U$392, U$421, U$44, U$450, U$479, U$508, U$537, U$566, U$595, U$624, U$653, U$682, U$73: device output:#RST_#1 -> output:##LP##2
- U$103, U$132, U$161, U$190, U$219, U$248, U$277, U$306, U$335, U$364, U$393, U$422, U$45, U$451, U$480, U$509, U$538, U$567, U$596, U$625, U$654, U$683, U$74: device output:##LP##2 -> output:#VDDA#0
- U$104, U$133, U$162, U$191, U$220, U$249, U$278, U$307, U$336, U$365, U$394, U$423, U$452, U$46, U$481, U$510, U$539, U$568, U$597, U$626, U$655, U$684, U$75: device output:#VDDA#0 -> output:#VDDIO#1
- U$105, U$134, U$163, U$192, U$221, U$250, U$279, U$308, U$337, U$366, U$395, U$424, U$453, U$47, U$482, U$511, U$540, U$569, U$598, U$627, U$656, U$685, U$76: device output:#VDDIO#1 -> output:VL53L5CX0
- U$106, U$135, U$164, U$193, U$222, U$251, U$280, U$309, U$338, U$367, U$396, U$425, U$454, U$48, U$483, U$512, U$541, U$570, U$599, U$628, U$657, U$686, U$77: device output:VL53L5CX0 -> output:IMAGER2
- U$107, U$136, U$165, U$194, U$223, U$252, U$281, U$310, U$339, U$368, U$397, U$426, U$455, U$484, U$49, U$513, U$542, U$571, U$600, U$629, U$658, U$687, U$78: device output:IMAGER2 -> output:TOF1
- U$108, U$137, U$166, U$195, U$224, U$253, U$282, U$311, U$340, U$369, U$398, U$427, U$456, U$485, U$50, U$514, U$543, U$572, U$601, U$630, U$659, U$688, U$79: device output:TOF1 -> output:#I�C#0
- U$109, U$138, U$167, U$196, U$225, U$254, U$283, U$312, U$341, U$370, U$399, U$428, U$457, U$486, U$51, U$515, U$544, U$573, U$602, U$631, U$660, U$689, U$80: device output:#I�C#0 -> output:#INT#1
- U$110, U$139, U$168, U$197, U$226, U$255, U$284, U$313, U$342, U$371, U$400, U$429, U$458, U$487, U$516, U$52, U$545, U$574, U$603, U$632, U$661, U$690, U$81: device output:#INT#1 -> output:#PSU#0
- U$111, U$140, U$169, U$198, U$227, U$256, U$285, U$314, U$343, U$372, U$401, U$430, U$459, U$488, U$517, U$53, U$546, U$575, U$604, U$633, U$662, U$691, U$82: device output:#PSU#0 -> output:VL53L5CX0
- U$112, U$141, U$170, U$199, U$228, U$257, U$286, U$315, U$344, U$373, U$402, U$431, U$460, U$489, U$518, U$54, U$547, U$576, U$605, U$634, U$663, U$692, U$83: device output:VL53L5CX0 -> output:TOF1
- U$113, U$142, U$171, U$200, U$229, U$258, U$287, U$316, U$345, U$374, U$403, U$432, U$461, U$490, U$519, U$548, U$55, U$577, U$606, U$635, U$664, U$693, U$84: device output:TOF1 -> output:IMAGER2
- U$114, U$143, U$172, U$201, U$230, U$259, U$288, U$317, U$346, U$375, U$404, U$433, U$462, U$491, U$520, U$549, U$56, U$578, U$607, U$636, U$665, U$694, U$85: device output:IMAGER2 -> output:#SCL#1
- U$115, U$144, U$173, U$202, U$231, U$260, U$289, U$318, U$347, U$376, U$405, U$434, U$463, U$492, U$521, U$550, U$57, U$579, U$608, U$637, U$666, U$695, U$86: device output:#SCL#1 -> output:#SDA#0
- U$116, U$145, U$174, U$203, U$232, U$261, U$290, U$319, U$348, U$377, U$406, U$435, U$464, U$493, U$522, U$551, U$58, U$580, U$609, U$638, U$667, U$696, U$87: device output:#SDA#0 -> output:ARD#0X290
- U$119, U$148, U$177, U$206, U$235, U$264, U$293, U$32, U$322, U$351, U$380, U$409, U$438, U$467, U$496, U$525, U$554, U$583, U$61, U$612, U$641, U$670, U$90: device output:ADR#0X520 -> output:#GND#62130
- U$120, U$149, U$178, U$207, U$236, U$265, U$294, U$323, U$33, U$352, U$381, U$410, U$439, U$468, U$497, U$526, U$555, U$584, U$613, U$62, U$642, U$671, U$91: device output:#GND#62130 -> output:#SDA#62131
- U$121, U$150, U$179, U$208, U$237, U$266, U$295, U$324, U$34, U$353, U$382, U$411, U$440, U$469, U$498, U$527, U$556, U$585, U$614, U$63, U$643, U$672, U$92: device output:#SDA#62131 -> output:#SCL#62132
- U$122, U$151, U$180, U$209, U$238, U$267, U$296, U$325, U$35, U$354, U$383, U$412, U$441, U$470, U$499, U$528, U$557, U$586, U$615, U$64, U$644, U$673, U$93: device output:#SCL#62132 -> output:#GND#62130
- U$123, U$152, U$181, U$210, U$239, U$268, U$297, U$326, U$355, U$36, U$384, U$413, U$442, U$471, U$500, U$529, U$558, U$587, U$616, U$645, U$65, U$674, U$94: device output:#GND#62130 -> output:#3V3#13
- U$125, U$154, U$183, U$212, U$241, U$270, U$299, U$328, U$357, U$38, U$386, U$415, U$444, U$473, U$502, U$531, U$560, U$589, U$618, U$647, U$67, U$676, U$96: device output:#3V3#13 -> output:PWR12
- U$126, U$155, U$184, U$213, U$242, U$271, U$300, U$329, U$358, U$387, U$39, U$416, U$445, U$474, U$503, U$532, U$561, U$590, U$619, U$648, U$677, U$68, U$97: device output:PWR12 -> output:#LED#10
- U$127, U$156, U$185, U$214, U$243, U$272, U$301, U$330, U$359, U$388, U$40, U$417, U$446, U$475, U$504, U$533, U$562, U$591, U$620, U$649, U$678, U$69, U$98: device output:#LED#10 -> output:#INT#0
- U$128, U$157, U$186, U$215, U$244, U$273, U$302, U$331, U$360, U$389, U$41, U$418, U$447, U$476, U$505, U$534, U$563, U$592, U$621, U$650, U$679, U$70, U$99: device output:#INT#0 -> output:#RST#1
- U$13: value (none) -> SFE_LOGO_NAME_FLAME.1_INCH; device output:ADR#0X520 -> SparkFun-Aesthetics:SFE_LOGO_NAME_FLAME_.1
- U$27: value SFE_LOGO_NAME_FLAME.1_INCH -> (none); device SparkFun-Aesthetics:SFE_LOGO_NAME_FLAME_.1 -> output:ARD#0X290
- moved U$254 19.1 mm to (54.4, 45.6)
- moved U$428 19.1 mm to (54.4, 71.5)
- moved U$602 19.1 mm to (54.4, 97.4)
- moved U$80 19.1 mm to (54.4, 19.7)
- moved U$196 19.1 mm to (2.54, 45.6)
- moved U$370 19.1 mm to (2.54, 71.5)
- moved U$544 19.1 mm to (2.54, 97.4)
- moved U$109 19.0 mm to (80.3, 19.7)
- moved U$138 19.0 mm to (106.2, 19.7)
- moved U$225 19.0 mm to (28.4, 45.6)
- moved U$283 19.0 mm to (80.3, 45.6)
- moved U$312 19.0 mm to (106.2, 45.6)
- moved U$399 19.0 mm to (28.4, 71.5)
- moved U$457 19.0 mm to (80.3, 71.5)
- moved U$486 19.0 mm to (106.2, 71.5)
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